File: rpi-industrial-analog.kicad_pcb (KiCad board)
At the start: 2 copper layers, 88.4 x 50 mm, 78 parts, among them J101 CONN_01X04, J102 CONN_01X08, U101 MCP3424, U102 ICL7660S A, U103 AD8220, U104 AD8220, U105 AD8220, U106 AD8220

Commit message: kicad version bump updating files
Parts:
- removed the ACC101 at (89.7, 123.7)
- removed the ACC105 at (89.7, 81.8)
Other:
- rule trace_min: 0.25 -> 0.13
- board text removed: "Frame Mounting Holes"
Changed lines of the file:
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@@
-(kicad_pcb (version 4) (host pcbnew 4.0.6)
+(kicad_pcb (version 4) (host pcbnew 4.0.7)
   (general
-    (links 150)
-    (no_connects 4)
-    (area 104.191999 77.902999 192.734001 128.091001)
+    (links 146)
+    (no_connects 0)
+    (area 86.424999 77.013 195.512 134.425)
     (thickness 1.6)
-    (drawings 35)
+    (drawings 34)
     (tracks 544)
     (zones 0)
-    (modules 78)
+    (modules 76)
     (nets 34)
   )
@@
     (zone_clearance 0.508)
     (zone_45_only no)
-    (trace_min 0.25)
+    (trace_min 0.13)
     (segment_width 0.2)
     (edge_width 0.15)
@@
     (mod_text_size 1 1)
     (mod_text_width 0.15)
-    (pad_size 3.2 3.2)
-    (pad_drill 3.2)
+    (pad_size 2 2)
+    (pad_drill 1.3)
     (pad_to_mask_clearance 0.0254)
     (solder_mask_min_width 0.1016)
@@
     (visible_elements 7FFFFF7F)
     (pcbplotparams
-      (layerselection 0x00008_00000000)
+      (layerselection 0x010fc_80000001)
       (usegerberextensions false)
       (excludeedgelayer true)
@@
       (drillshape 0)
       (scaleselection 1)
-      (outputdirectory /Users/davisjp/Desktop/OshStencils/))
+      (outputdirectory C:/Users/davisjp/Desktop/ap-macrofab/))
   )
   (net 0 "")
@@
     (add_net "Net-(R102-Pad2)")
   )
-  (module Mounting_Holes:MountingHole_3.2mm_M3_DIN965 (layer F.Cu)
-    (at 89.725 123.698)
-    (descr "Mounting Hole 3.2mm, no annular, M3, DIN965")
-    (tags "mounting hole 3.2mm no annular m3 din965")
-    (fp_text reference ACC101 (at 0 -3.8) (layer F.SilkS) hide
-      (effects (font (size 1 1) (thickness 0.15)))
-    )
-    (fp_text value ACC_? (at 0 3.8) (layer F.Fab)
-      (effects (font (size 1 1) (thickness 0.15)))
-    )
-    (fp_circle (center 0 0) (end 2.8 0) (layer Cmts.User) (width 0.15))
-    (fp_circle (center 0 0) (end 3.05 0) (layer F.CrtYd) (width 0.05))
-    (pad "" np_thru_hole circle (at 0 0) (size 3.2 3.2) (drill 3.2) (layers *.Cu *.Mask F.Paste))
-  )
-  (module Mounting_Holes:MountingHole_3.2mm_M3_DIN965 (layer F.Cu)
-    (at 89.7 81.825)
-    (descr "Mounting Hole 3.2mm, no annular, M3, DIN965")
-    (tags "mounting hole 3.2mm no annular m3 din965")
-    (fp_text reference ACC105 (at 0 -3.8) (layer F.SilkS) hide
-      (effects (font (size 1 1) (thickness 0.15)))
-    )
-    (fp_text value ACC_? (at 0 3.8) (layer F.Fab)
-      (effects (font (size 1 1) (thickness 0.15)))
-    )
-    (fp_circle (center 0 0) (end 2.8 0) (layer Cmts.User) (width 0.15))
-    (fp_circle (center 0 0) (end 3.05 0) (layer F.CrtYd) (width 0.05))
-    (pad "" np_thru_hole circle (at 0 0) (size 3.2 3.2) (drill 3.2) (layers *.Cu *.Mask F.Paste))
-  )
   (module GRPB031VWTC-RC_3pos_Header (layer F.Cu)
     (at 144.653 87.122 270)
@@
     (pad 6 thru_hole circle (at 20 0 90) (size 2 2) (drill 1.3) (layers *.Cu *.Mask)
       (net 11 /AIN3-))
-    (pad 5 thru_hole circle (at 15 0 90) (size 2 2) (drill 1.3) (layers *.Cu *.Mask F.Paste)
+    (pad 5 thru_hole circle (at 15 0 90) (size 2 2) (drill 1.3) (layers *.Cu *.Mask)
       (net 16 /AIN3+))
     (pad 2 thru_hole circle (at 0 0 90) (size 2 2) (drill 1.3) (layers *.Cu *.Mask)
@@
       (xy 0.633952 -5.96402) (xy 0.746535 -5.366828)) (layer F.SilkS) (width 0.01))
   )
-  (gr_text "Frame Mounting Holes" (at 89.675 101.975 90) (layer F.SilkS)
-    (effects (font (size 1.5 1.5) (thickness 0.3)))
-  )
   (gr_text - (at 183.05 85.75) (layer F.SilkS)
