File: rpi-industrial-analog.sch (KiCad schematic (older format))
At the start: 80 parts, among them J101 CONN_01X04, J102 CONN_01X08, U101 MCP3424, U102 ICL7660S A, U103 AD8220, U104 AD8220, U105 AD8220, U106 AD8220

Commit message: schematic library switched to master library
Parts:
- D107, D108, D109, D110: symbol TVS_Small -> D_TVS_ALT; Populate (none) -> 1
- U104: Populate (none) -> 1
Changed lines of the file:
@@
 EESchema Schematic File Version 2
-LIBS:raspberrypi_2_b
-LIBS:3ML_LLC_Component_Library
 LIBS:power
 LIBS:device
@@
 LIBS:contrib
 LIBS:valves
+LIBS:3ML_AnalogDevices
+LIBS:3ML_Microchip
+LIBS:3ML_Texas_Instruments
 LIBS:rpi-industrial-analog-cache
 EELAYER 25 0
@@
 $EndComp
 $Comp
-L TVS_Small D107
+L D_TVS_ALT D107
 U 1 1 58D89DB3
 P 8350 1750
@@
 F 2 "3ML_Footprint_Library:DO-214AA_Hand_Soldering" H 8350 1750 50  0001 C CNN
 F 3 "http://www.littelfuse.com/~/media/electronics/datasheets/tvs_diodes/littelfuse_tvs_diode_smbj_datasheet.pdf.pdf" H 8350 1750 50  0001 C CNN
-F 4 "SMBJ20CALFCT-ND" H 8350 1750 60  0001 C CNN "MPN"
-F 5 "Littelfuse Inc" H 8350 1750 60  0001 C CNN "MFN"
-F 6 "X" H 8350 1750 60  0001 C CNN "Characteristics"
-F 7 "TVS Diode" H 8350 1750 60  0001 C CNN "Description"
-F 8 "DO-214AA" H 8350 1750 60  0001 C CNN "Package ID"
-F 9 "Digikey" H 8350 1750 60  0001 C CNN "Source"
-F 10 "Y" H 8350 1750 60  0001 C CNN "Critical"
-F 11 "X" H 8350 1750 60  0001 C CNN "Notes"
+F 4 "X" H 8350 1750 60  0001 C CNN "Characteristics"
+F 5 "TVS Diode" H 8350 1750 60  0001 C CNN "Description"
+F 6 "Littelfuse Inc" H 8350 1750 60  0001 C CNN "MFN"
+F 7 "DO-214AA" H 8350 1750 60  0001 C CNN "Package ID"
+F 8 "Digikey" H 8350 1750 60  0001 C CNN "Source"
+F 9 "Y" H 8350 1750 60  0001 C CNN "Critical"
+F 10 "X" H 8350 1750 60  0001 C CNN "Notes"
+F 11 "1" H 8350 1750 60  0001 C CNN "Populate"
+F 12 "SMBJ20CALFCT-ND" H 8350 1750 60  0001 C CNN "MPN"
 	1    8350 1750
 	0    1    1    0
@@
 F 2 "Housings_SSOP:MSOP-8_3x3mm_Pitch0.65mm" H 6500 3700 60  0001 C CNN
 F 3 "http://www.analog.com/media/en/technical-documentation/data-sheets/AD8220.pdf" H 6500 3700 60  0001 C CNN
-F 4 "AD8220ARMZ" H 6500 3700 60  0001 C CNN "MPN"
-F 5 "Analog Devices Inc" H 6500 3700 60  0001 C CNN "MFN"
-F 6 "X" H 6500 3700 60  0001 C CNN "Characteristics"
-F 7 "Instrumentation Amplifier 1 Circuit Rail-to-Rail 8-MSOP" H 6500 3700 60  0001 C CNN "Description"
-F 8 "8-TSSOP" H 6500 3700 60  0001 C CNN "Package ID"
-F 9 "Digikey" H 6500 3700 60  0001 C CNN "Source"
-F 10 "Y" H 6500 3700 60  0001 C CNN "Critical"
-F 11 "X" H 6500 3700 60  0001 C CNN "Notes"
+F 4 "X" H 6500 3700 60  0001 C CNN "Characteristics"
+F 5 "Instrumentation Amplifier 1 Circuit Rail-to-Rail 8-MSOP" H 6500 3700 60  0001 C CNN "Description"
+F 6 "Analog Devices Inc" H 6500 3700 60  0001 C CNN "MFN"
+F 7 "8-TSSOP" H 6500 3700 60  0001 C CNN "Package ID"
+F 8 "Digikey" H 6500 3700 60  0001 C CNN "Source"
+F 9 "Y" H 6500 3700 60  0001 C CNN "Critical"
+F 10 "X" H 6500 3700 60  0001 C CNN "Notes"
+F 11 "1" H 6500 3700 60  0001 C CNN "Populate"
+F 12 "AD8220ARMZ" H 6500 3700 60  0001 C CNN "MPN"
 	1    6500 3700
 	-1   0    0    -1
@@
 NoConn ~ 7000 3700
 $Comp
-L TVS_Small D108
+L D_TVS_ALT D108
 U 1 1 58D89117
 P 8350 3600
@@
 F 2 "3ML_Footprint_Library:DO-214AA_Hand_Soldering" H 8350 3600 50  0001 C CNN
 F 3 "http://www.littelfuse.com/~/media/electronics/datasheets/tvs_diodes/littelfuse_tvs_diode_smbj_datasheet.pdf.pdf" H 8350 3600 50  0001 C CNN
-F 4 "SMBJ20CALFCT-ND" H 8350 3600 60  0001 C CNN "MPN"
-F 5 "Littelfuse Inc" H 8350 3600 60  0001 C CNN "MFN"
-F 6 "X" H 8350 3600 60  0001 C CNN "Characteristics"
-F 7 "TVS Diode" H 8350 3600 60  0001 C CNN "Description"
-F 8 "DO-214AA" H 8350 3600 60  0001 C CNN "Package ID"
-F 9 "Digikey" H 8350 3600 60  0001 C CNN "Source"
-F 10 "Y" H 8350 3600 60  0001 C CNN "Critical"
-F 11 "X" H 8350 3600 60  0001 C CNN "Notes"
+F 4 "X" H 8350 3600 60  0001 C CNN "Characteristics"
+F 5 "TVS Diode" H 8350 3600 60  0001 C CNN "Description"
+F 6 "Littelfuse Inc" H 8350 3600 60  0001 C CNN "MFN"
+F 7 "DO-214AA" H 8350 3600 60  0001 C CNN "Package ID"
+F 8 "Digikey" H 8350 3600 60  0001 C CNN "Source"
+F 9 "Y" H 8350 3600 60  0001 C CNN "Critical"
+F 10 "X" H 8350 3600 60  0001 C CNN "Notes"
+F 11 "1" H 8350 3600 60  0001 C CNN "Populate"
+F 12 "SMBJ20CALFCT-ND" H 8350 3600 60  0001 C CNN "MPN"
 	1    8350 3600
 	0    1    1    0
@@
 NoConn ~ 7000 5550
 $Comp
-L TVS_Small D109
+L D_TVS_ALT D109
 U 1 1 58D89636
 P 8350 5450
@@
 F 2 "3ML_Footprint_Library:DO-214AA_Hand_Soldering" H 8350 5450 50  0001 C CNN
 F 3 "http://www.littelfuse.com/~/media/electronics/datasheets/tvs_diodes/littelfuse_tvs_diode_smbj_datasheet.pdf.pdf" H 8350 5450 50  0001 C CNN
-F 4 "SMBJ20CALFCT-ND" H 8350 5450 60  0001 C CNN "MPN"
-F 5 "Littelfuse Inc" H 8350 5450 60  0001 C CNN "MFN"
-F 6 "X" H 8350 5450 60  0001 C CNN "Characteristics"
-F 7 "TVS Diode" H 8350 5450 60  0001 C CNN "Description"
-F 8 "DO-214AA" H 8350 5450 60  0001 C CNN "Package ID"
-F 9 "Digikey" H 8350 5450 60  0001 C CNN "Source"
-F 10 "Y" H 8350 5450 60  0001 C CNN "Critical"
-F 11 "X" H 8350 5450 60  0001 C CNN "Notes"
+F 4 "X" H 8350 5450 60  0001 C CNN "Characteristics"
+F 5 "TVS Diode" H 8350 5450 60  0001 C CNN "Description"
+F 6 "Littelfuse Inc" H 8350 5450 60  0001 C CNN "MFN"
+F 7 "DO-214AA" H 8350 5450 60  0001 C CNN "Package ID"
+F 8 "Digikey" H 8350 5450 60  0001 C CNN "Source"
+F 9 "Y" H 8350 5450 60  0001 C CNN "Critical"
+F 10 "X" H 8350 5450 60  0001 C CNN "Notes"
+F 11 "1" H 8350 5450 60  0001 C CNN "Populate"
+F 12 "SMBJ20CALFCT-ND" H 8350 5450 60  0001 C CNN "MPN"
 	1    8350 5450
 	0    1    1    0
@@
 NoConn ~ 7000 7150
 $Comp
-L TVS_Small D110
+L D_TVS_ALT D110
 U 1 1 58D8972D
 P 8350 7050
@@
 F 2 "3ML_Footprint_Library:DO-214AA_Hand_Soldering" H 8350 7050 50  0001 C CNN
 F 3 "http://www.littelfuse.com/~/media/electronics/datasheets/tvs_diodes/littelfuse_tvs_diode_smbj_datasheet.pdf.pdf" H 8350 7050 50  0001 C CNN
-F 4 "SMBJ20CALFCT-ND" H 8350 7050 60  0001 C CNN "MPN"
-F 5 "Littelfuse Inc" H 8350 7050 60  0001 C CNN "MFN"
-F 6 "X" H 8350 7050 60  0001 C CNN "Characteristics"
-F 7 "TVS Diode" H 8350 7050 60  0001 C CNN "Description"
-F 8 "DO-214AA" H 8350 7050 60  0001 C CNN "Package ID"
-F 9 "Digikey" H 8350 7050 60  0001 C CNN "Source"
-F 10 "Y" H 8350 7050 60  0001 C CNN "Critical"
-F 11 "X" H 8350 7050 60  0001 C CNN "Notes"
+F 4 "X" H 8350 7050 60  0001 C CNN "Characteristics"
+F 5 "TVS Diode" H 8350 7050 60  0001 C CNN "Description"
+F 6 "Littelfuse Inc" H 8350 7050 60  0001 C CNN "MFN"
+F 7 "DO-214AA" H 8350 7050 60  0001 C CNN "Package ID"
+F 8 "Digikey" H 8350 7050 60  0001 C CNN "Source"
+F 9 "Y" H 8350 7050 60  0001 C CNN "Critical"
+F 10 "X" H 8350 7050 60  0001 C CNN "Notes"
+F 11 "1" H 8350 7050 60  0001 C CNN "Populate"
+F 12 "SMBJ20CALFCT-ND" H 8350 7050 60  0001 C CNN "MPN"
 	1    8350 7050
 	0    1    1    0
@@
 Connection ~ 8650 2000
 Wire Wire Line
-	8350 1950 8350 2000
+	8350 1900 8350 2000
 Connection ~ 8350 2000
 Connection ~ 8350 1550
@@
 Connection ~ 8650 3850
 Wire Wire Line
-	8350 3800 8350 3850
+	8350 3750 8350 3850
 Connection ~ 8350 3850
 Connection ~ 8350 3400
@@
 Connection ~ 8650 5700
 Wire Wire Line
-	8350 5650 8350 5700
+	8350 5600 8350 5700
 Connection ~ 8350 5700
 Connection ~ 8350 5250
@@
 Connection ~ 8650 7300
 Wire Wire Line
-	8350 7250 8350 7300
+	8350 7200 8350 7300
 Connection ~ 8350 7300
 Connection ~ 8350 6850
@@
 	1    0    0    -1
 $EndComp
+Wire Wire Line
+	8350 1550 8350 1600
+Wire Wire Line
+	8350 3400 8350 3450
+Wire Wire Line
+	8350 5250 8350 5300
+Wire Wire Line
+	8350 6850 8350 6900
 $EndSCHEMATC

Commit message: updating footprints to use master library
Parts:
- J102: footprint 3ML_Footprint_Library:1935226 -> 3ML_Conn_Headers:Phoenix-1x8-1935226; Populate (none) -> 1
- JP101, JP102, JP103, JP104: footprint 3ML_Footprint_Library:GRPB031VWTC-RC_3pos_Header -> 3ML_Conn_Headers:Sullins-1x3-Jumper-GRPB031VWTC-RC; Populate (none) -> 1
- TP103, TP104, TP105, TP106: footprint 3ML_Footprint_Library:Keystone_5000_Test_Point_Mini -> 3ML_Test_Points:Keystone_5000_Test_Point_Mini; Populate (none) -> 1

Commit message: kicad version bump updating files
Parts:
- C106: MPN (none) -> F931A106KAA
- U101: symbol MCP3424 -> MCP3424-RESCUE-rpi-industrial-analog
Changed lines of the file:
@@
 EESchema Schematic File Version 2
+LIBS:rpi-industrial-analog-rescue
 LIBS:power
 LIBS:device
@@
 $EndComp
 $Comp
-L MCP3424 U101
+L MCP3424-RESCUE-rpi-industrial-analog U101
 U 1 1 58D81EDC
 P 2250 2850
@@
 F 2 "Capacitors_Tantalum_SMD:CP_Tantalum_Case-A_EIA-3216-18_Reflow" H 1550 5150 50  0001 C CNN
 F 3 "http://datasheets.avx.com/F93.pdf" H 1550 5150 50  0001 C CNN
-F 4 "X" H 1550 5150 60  0001 C CNN "Characteristics"
-F 5 "F931A106KAA" H 1550 5150 60  0001 C CNN "Description"
-F 6 "AVX Corporation" H 1550 5150 60  0001 C CNN "MFN"
-F 7 "1206 (3216 Metric)" H 1550 5150 60  0001 C CNN "Package ID"
-F 8 "Digikey" H 1550 5150 60  0001 C CNN "Source"
-F 9 "Y" H 1550 5150 60  0001 C CNN "Critical"
-F 10 "X" H 1550 5150 60  0001 C CNN "Notes"
-F 11 "1" H 1550 5150 60  0001 C CNN "Populate"
+F 4 "F931A106KAA" H 1550 5150 60  0001 C CNN "MPN"
+F 5 "AVX Corporation" H 1550 5150 60  0001 C CNN "MFN"
+F 6 "X" H 1550 5150 60  0001 C CNN "Characteristics"
+F 7 "F931A106KAA" H 1550 5150 60  0001 C CNN "Description"
+F 8 "1206 (3216 Metric)" H 1550 5150 60  0001 C CNN "Package ID"
+F 9 "Digikey" H 1550 5150 60  0001 C CNN "Source"
+F 10 "Y" H 1550 5150 60  0001 C CNN "Critical"
+F 11 "X" H 1550 5150 60  0001 C CNN "Notes"
+F 12 "1" H 1550 5150 60  0001 C CNN "Populate"
 	1    1550 5150
 	1    0    0    -1
